File: schematics/remmy_rf_mouse/remmy_rf_mouse.kicad_sch (KiCad schematic)
At the start: 72 parts, among them IC1 MP2667GG-0000-Z, IC2 NRF54L15-QFAA-R, IC3 PMW3360DM-T2QU, IC4 ISL9120IR, IC5 TPS73219DBVT, IC6 AP2112K-3.3TRG1, J1 USB_C_Receptacle_USB2.0_14P, J2 Conn_01x03_Pin, J3 PH2.0, J4 Conn_ARM_JTAG_SWD_10, J5 U.FL-R-SMT_10_, Q1 BSS138, SW1 RotaryEncoder, SW2 Kailh GM 8.0, SW3 Kailh GM 8.0, SW4 SW_Push, SW5 SW_Push, SW6 SW_Push, X1 ABS06-32.768KHZ-9-T, Y1 Crystal_GND24

Commit message: fixed most footprints, just matching network left
Parts:
- removed C13: 10u, Capacitor_SMD:C_0805_2012Metric_Pad1.18x1.45mm_HandSolder, symbol Device:C
- removed IC3: PMW3360DM-T2QU, Custom_FP:PMW3360DM-T2QU, symbol Custom_sym:PMW3360DM-T2QU
- removed Q1: BSS138, Package_TO_SOT_SMD:SOT-23, symbol Transistor_FET:BSS138
- removed R1, R2, R5, R7: 10k, Resistor_SMD:R_0402_1005Metric_Pad0.72x0.64mm_HandSolder, symbol Device:R
- added IC2: PMW3395DM-T6QU, Custom_FP:PMW3360DM-T2QU, symbol Custom_sym:PMW3395DM-T6QU
- added R3: 10k, Resistor_SMD:R_0402_1005Metric_Pad0.72x0.64mm_HandSolder, symbol Device:R
- added TP1, TP2, TP3, TP4, TP5, TP6, TP7: TestPoint, TestPoint:TestPoint_Pad_D1.0mm, symbol Connector:TestPoint
- C11: renamed from C24; value 0.1u -> 100n
- C12: renamed from C14; value 0.1u -> 33u; footprint Capacitor_SMD:C_0402_1005Metric_Pad0.74x0.62mm_HandSolder -> Capacitor_SMD:C_0805_2012Metric_Pad1.18x1.45mm_HandSolder
- C13: renamed from C1; footprint Capacitor_SMD:C_0402_1005Metric_Pad0.74x0.62mm_HandSolder -> Capacitor_SMD:C_0603_1608Metric_Pad1.08x0.95mm_HandSolder
- C20: renamed from C21; footprint Capacitor_SMD:C_0201_0603Metric_Pad0.64x0.40mm_HandSolder -> (none)
- C22: renamed from C25; footprint Capacitor_SMD:C_0201_0603Metric_Pad0.64x0.40mm_HandSolder -> (none)
- C25: renamed from C30; footprint Capacitor_SMD:C_0402_1005Metric_Pad0.74x0.62mm_HandSolder -> (none)
- C4: renamed from C15; value 0.1u -> 100n
- C5: renamed from C28; value 0.1u -> 100n
- C7: renamed from C5; footprint (none) -> Capacitor_SMD:C_0603_1608Metric_Pad1.08x0.95mm_HandSolder
- C8: renamed from C2; footprint Capacitor_SMD:C_0402_1005Metric_Pad0.74x0.62mm_HandSolder -> Capacitor_SMD:C_0603_1608Metric_Pad1.08x0.95mm_HandSolder
- C9: renamed from C6; footprint (none) -> Capacitor_SMD:C_0805_2012Metric_Pad1.18x1.45mm_HandSolder
- FB1: footprint Capacitor_SMD:C_0201_0603Metric_Pad0.64x0.40mm_HandSolder -> Inductor_SMD:L_0201_0603Metric_Pad0.64x0.40mm_HandSolder
- IC1: renamed from IC4; footprint (none) -> Custom_FP:QFN-12-1EP_3x3mm_P0.5mm_EP1.45x1.45mm
- IC3: renamed from IC1; footprint (none) -> Imported_FP:QFN-10_2mmx2mm_MNP
- L1: footprint (none) -> Custom_FP:L_Bourns-SRN2010
- L2, L3, L5: footprint Inductor_SMD:L_0201_0603Metric_Pad0.64x0.40mm_HandSolder -> (none)
- R1: renamed from R9; footprint Resistor_SMD:R_0402_1005Metric_Pad0.72x0.64mm_HandSolder -> Resistor_SMD:R_0603_1608Metric_Pad0.98x0.95mm_HandSolder
- R2: renamed from R10; footprint Resistor_SMD:R_0402_1005Metric_Pad0.72x0.64mm_HandSolder -> Resistor_SMD:R_0603_1608Metric_Pad0.98x0.95mm_HandSolder
- R4: renamed from R12; footprint (none) -> Resistor_SMD:R_0402_1005Metric_Pad0.72x0.64mm_HandSolder
- R5: renamed from R13; footprint (none) -> Resistor_SMD:R_0402_1005Metric_Pad0.72x0.64mm_HandSolder
- R8: renamed from R11; footprint Resistor_SMD:R_0402_1005Metric_Pad0.72x0.64mm_HandSolder -> Resistor_SMD:R_0603_1608Metric_Pad0.98x0.95mm_HandSolder
- R9: renamed from R6; value 39 -> 5.6; footprint Resistor_SMD:R_0402_1005Metric_Pad0.72x0.64mm_HandSolder -> Resistor_SMD:R_0603_1608Metric_Pad0.98x0.95mm_HandSolder
- X1: footprint ABS06-32.768KHZ-9-T:XTAL_ABS06-32.768KHZ-9-T -> Imported_FP:XTAL_ABS06-32.768KHZ-9-T; now not fitted
- renumbered C4 to C1, C22 to C10, C3 to C14, C12 to C15, C18 to C17, C19 to C18, C20 to C19, C7 to C2, C23 to C21, C26 to C23, C27 to C24, C31 to C26, C32 to C27, C29 to C3, C17 to C6, IC6 to IC4, IC2 to IC6, J3 to J2, J2 to J3, JP4 to JP2, JP5 to JP3, JP2 to JP4, R4 to R10, R3 to R6, R8 to R7, SW2 to SW1, SW3 to SW2, SW1 to SW3
Connections:
- net +1.9V: now also R9.2, IC2.4 (VDD); no longer R9.1
- net +3.3V: now also IC2.7 (VDDIO), R3.1
- net +3.6V: now also D1.4 (VDD)
- net ARGB: now also D1.3 (DIN)
- net DPI: now also IC6.27 (P0.02); no longer IC6.8 (P1.07/ASI(1)/AIN3)
- net ENC_A: now also IC6.7 (P1.06/ASO(1)/AIN2); no longer IC6.37 (P1.09/ASO(2)/RADIO(0))
- net ENC_B: now also IC6.8 (P1.07/ASI(1)/AIN3); no longer IC6.38 (P1.10/ASI(2)/RADIO(1))
- net GND: now also IC2.3 (GND), IC2.8 (GNDIO)
- net I2C_SCL: now also TP6.1
- net I2C_SDA: now also TP7.1
- net MOTION: now also IC6.42 (P1.14/RADIO(5)/AIN7), IC2.9 (MOTION), TP5.1; no longer IC6.40 (P1.12/ASI(3)/RADIO(3)/AIN5)
- net MOUSE1: now also IC6.9 (P1.08/CLK16M/EXTREF); no longer IC6.3 (P1.02/NFC1)
- net MOUSE2: now also IC6.5 (P1.04/ASO(0)/AIN0); no longer IC6.4 (P1.03/NFC2)
- net MOUSE4: now also IC6.4 (P1.03/NFC2); no longer IC6.6 (P1.05/ASI(0)/RADIO(6)/AIN1)
- net MOUSE5: now also IC6.3 (P1.02/NFC1); no longer IC6.7 (P1.06/ASO(1)/AIN2)
- net SPI_CLK: now also IC6.41 (P1.13/RADIO(4)/AIN6), IC2.10 (SCLK), TP4.1; no longer IC6.39 (P1.11/ASO(3)/RADIO(2)/AIN4)
- net SPI_MISO: now also IC6.39 (P1.11/ASO(3)/RADIO(2)/AIN4), IC2.12 (MISO), R3.2, TP2.1; no longer IC6.42 (P1.14/RADIO(5)/AIN7)
- net SPI_MOSI: now also IC6.40 (P1.12/ASI(3)/RADIO(3)/AIN5), IC2.11 (MOSI), TP3.1; no longer IC6.41 (P1.13/RADIO(4)/AIN6)
- net SPI_NCS: now also IC6.38 (P1.10/ASI(2)/RADIO(1)), IC2.13 (NCS), TP1.1; no longer IC6.9 (P1.08/CLK16M/EXTREF)
- net nRESET: no longer C15.1, IC6.30 (~{RESET}), R10.2, SW6.2
- net at C3.1, C5.1: now also IC2.5 (VDDREG)
- net MWHEEL_BUTTON renamed MOUSE3
- net MOUSE3: now also IC6.6 (P1.05/ASI(0)/RADIO(6)/AIN1); no longer IC6.5 (P1.04/ASO(0)/AIN0)
- new net: IC2.15 (LED_P), R9.1
- new net NRST: C15.1, IC6.30 (~{RESET}), R10.2, SW6.2
- new net SENSOR_NRST: IC2.14 (NRESET), IC6.37 (P1.09/ASO(2)/RADIO(0))
- no-connect marks 18 -> 17
Other:
- note added: "OPTICAL SENSOR - PMW3395"
- note removed: "OPTICAL SENSOR - PMW3360"
- moved on the sheet: C10, C11, C12, C3, C4, C5, C6, D1, J3, R9, SW4, SW6
